Commit message: restructure arguments and indentations

File: config/srdf/tiago_pro.srdf.xacro (robot description, xacro)
@@ -4,26 +4,27 @@
     A URDF file must exist for this robot as well, where the joints and the links that are referenced are defined
 -->
-<robot name="tiago_pro" xmlns:xacro="http://ros.org/wiki/xacro">
+<robot name="tiago_pro"
+    xmlns:xacro="http://ros.org/wiki/xacro">
     <xacro:arg name="arm_type_left" default="tiago-arm"/>
+    <xacro:arg name="arm_type_right" default="tiago-arm"/>
     <xacro:arg name="end_effector_left" default="pal-hey5"/>
+    <xacro:arg name="end_effector_right" default="pal-hey5"/>
     <xacro:arg name="ft_sensor_left" default="rokubi"/>
+    <xacro:arg name="ft_sensor_right" default="rokubi"/>
     <xacro:property name="arm_type_left" value="$(arg arm_type_left)"/>
+    <xacro:property name="arm_type_right" value="$(arg arm_type_right)"/>
+    <xacro:property name="has_arm_right" value="${arm_type_right not in ['no-arm']}"/>
     <xacro:property name="has_arm_left" value="${arm_type_left not in ['no-arm']}"/>
     <xacro:property name="end_effector_left" value="$(arg end_effector_left)"/>
+    <xacro:property name="end_effector_left_arg" value="$(arg end_effector_left)"/>
+    <xacro:property name="end_effector_right" value="$(arg end_effector_right)"/>
+    <xacro:property name="end_effector_right_arg" value="$(arg end_effector_right)"/>
     <xacro:property name="ft_sensor_left" value="$(arg ft_sensor_left)"/>
+    <xacro:property name="ft_sensor_right" value="$(arg ft_sensor_right)"/>
     <xacro:property name="has_ft_sensor_left" value="${ft_sensor_left not in ['no-ft-sensor']}"/>
-    <xacro:arg name="arm_type_right" default="tiago-arm"/>
-    <xacro:arg name="end_effector_right" default="pal-hey5"/>
-    <xacro:arg name="ft_sensor_right" default="rokubi"/>
-    <xacro:property name="arm_type_right" value="$(arg arm_type_right)"/>
-    <xacro:property name="has_arm_right" value="${arm_type_right not in ['no-arm']}"/>
-    <xacro:property name="end_effector_right" value="$(arg end_effector_right)"/>
-    <xacro:property name="ft_sensor_right" value="$(arg ft_sensor_right)"/>
     <xacro:property name="has_ft_sensor_right" value="${ft_sensor_right not in ['no-ft-sensor']}"/>
     <!-- https://answers.ros.org/question/276062/adding-objects-in-moveit-fixed-in-the-world-while-the-mobile-manipulator-is-moving-confusion-with-root_joint-planning_frame-and-srdf-structure/ -->
+    <xacro:property name="robot" value="tiago_pro"/>
     <virtual_joint name="odom_to_base" child_link="base_footprint" parent_frame="odom" type="planar"/>
-    <xacro:property name="robot" value="tiago_pro"/>
-    <xacro:property name="end_effector_left_arg" value="$(arg end_effector_left)"/>
-    <xacro:property name="end_effector_right_arg" value="$(arg end_effector_right)"/>
     <xacro:if value="${end_effector_left == 'no-end-effector'}">
         <xacro:property name="end_effector_left_arg" value="no-ee"/>
@@ -37,33 +38,33 @@
     <!--CHAINS: When a chain is specified, all the links along the chain (including endpoints) are included in the group. Additionally, all the joints that are parents to included links are also included. This means that joints along the chain and the parent joint of the base link are included in the group-->
     <!--SUBGROUPS: Groups can also be formed by referencing to already defined group names-->
-<xacro:macro name="arm_groups" params="side">
-    <group name="arm_${side}">
-        <joint name="arm_${side}_1_joint" />
-        <joint name="arm_${side}_2_joint" />
-        <joint name="arm_${side}_3_joint" />
-        <joint name="arm_${side}_4_joint" />
-        <joint name="arm_${side}_5_joint" />
-        <joint name="arm_${side}_6_joint" />
-        <joint name="arm_${side}_7_joint" />
-        <joint name="arm_${side}_tool_joint" />
-    </group>
-    <group name="arm_${side}_torso">
-        <group name="arm_${side}" />
-        <group name="torso" />
-    </group>
-</xacro:macro>
-<xacro:if value="${has_arm_left}">
-<xacro:arm_groups side="left"/>
-</xacro:if>
-<xacro:if value="${has_arm_right}">
-<xacro:arm_groups side="right"/>
-</xacro:if>
-<xacro:if value="${has_arm_left and has_arm_right}">
-    <group name="both_arms_torso">
-        <group name="torso" />
-        <group name="arm_right" />
-        <group name="arm_left" />
-    </group>
-</xacro:if>
+    <xacro:macro name="arm_groups" params="side">
+        <group name="arm_${side}">
+            <joint name="arm_${side}_1_joint" />
+            <joint name="arm_${side}_2_joint" />
+            <joint name="arm_${side}_3_joint" />
+            <joint name="arm_${side}_4_joint" />
+            <joint name="arm_${side}_5_joint" />
+            <joint name="arm_${side}_6_joint" />
+            <joint name="arm_${side}_7_joint" />
+            <joint name="arm_${side}_tool_joint" />
+        </group>
+        <group name="arm_${side}_torso">
+            <group name="arm_${side}" />
+            <group name="torso" />
+        </group>
+    </xacro:macro>
+    <xacro:if value="${has_arm_left}">
+        <xacro:arm_groups side="left"/>
+    </xacro:if>
+    <xacro:if value="${has_arm_right}">
+        <xacro:arm_groups side="right"/>
+    </xacro:if>
+    <xacro:if value="${has_arm_left and has_arm_right}">
+        <group name="both_arms_torso">
+            <group name="torso" />
+            <group name="arm_right" />
+            <group name="arm_left" />
+        </group>
+    </xacro:if>
     <group name="torso">
         <joint name="torso_lift_joint" />
@@ -71,30 +72,30 @@
     <xacro:macro name="end_effector_for_side" params="side end_effector">
         <xacro:include filename="$(find pal_sea_arm_moveit_config)/config/srdf/end_effectors/${end_effector}.srdf.xacro" />
-    <xacro:define_end_effector arm="arm_${side}" name="${end_effector_name}_${side}"/>
-</xacro:macro>
-<xacro:if value="${has_arm_left}">
-    <xacro:end_effector_for_side side="left" end_effector="${end_effector_left}"/>
-    <xacro:if value="${has_ft_sensor_left}">
-        <xacro:property name="config_left" value="${end_effector_left_arg}_${ft_sensor_left}"/>
+        <xacro:define_end_effector arm="arm_${side}" name="${end_effector_name}_${side}"/>
+    </xacro:macro>
+    <xacro:if value="${has_arm_left}">
+        <xacro:end_effector_for_side side="left" end_effector="${end_effector_left}"/>
+        <xacro:if value="${has_ft_sensor_left}">
+            <xacro:property name="config_left" value="${end_effector_left_arg}_${ft_sensor_left}"/>
+        </xacro:if>
+        <xacro:unless value="${has_ft_sensor_left}">
+            <xacro:property name="config_left" value="${end_effector_left_arg}"/>
+        </xacro:unless>
     </xacro:if>
-    <xacro:unless value="${has_ft_sensor_left}">
-        <xacro:property name="config_left" value="${end_effector_left_arg}"/>
+    <xacro:unless value="${has_arm_left}">
+        <xacro:property name="config_left" value="no-arm-left"/>
     </xacro:unless>
-</xacro:if>
-<xacro:unless value="${has_arm_left}">
-    <xacro:property name="config_left" value="no-arm-left"/>
-</xacro:unless>
-<xacro:if value="${has_arm_right}">
-    <xacro:end_effector_for_side side="right" end_effector="${end_effector_right}"/>
-    <xacro:if value="${has_ft_sensor_right}">
-        <xacro:property name="config_right" value="${end_effector_right_arg}_${ft_sensor_right}"/>
+    <xacro:if value="${has_arm_right}">
+        <xacro:end_effector_for_side side="right" end_effector="${end_effector_right}"/>
+        <xacro:if value="${has_ft_sensor_right}">
+            <xacro:property name="config_right" value="${end_effector_right_arg}_${ft_sensor_right}"/>
+        </xacro:if>
+        <xacro:unless value="${has_ft_sensor_right}">
+            <xacro:property name="config_right" value="${end_effector_right_arg}"/>
+        </xacro:unless>
     </xacro:if>
-    <xacro:unless value="${has_ft_sensor_right}">
-        <xacro:property name="config_right" value="${end_effector_right_arg}"/>
+    <xacro:unless value="${has_arm_right}">
+        <xacro:property name="config_right" value="no-arm-right"/>
     </xacro:unless>
-</xacro:if>
-<xacro:unless value="${has_arm_right}">
-    <xacro:property name="config_right" value="no-arm-right"/>
-</xacro:unless>
-<xacro:include filename="$(find tiago_pro_moveit_config)/config/srdf/disable_collisions/${robot}_${config_left}_${config_right}.srdf.xacro" />
+    <xacro:include filename="$(find tiago_pro_moveit_config)/config/srdf/disable_collisions/${robot}_${config_left}_${config_right}.srdf.xacro" />
 </robot>
